Commit message: Add files via upload

File: ur5/urdf/ur5_joint_limited_robot.urdf.xacro (robot description, xacro)
@@ -9,5 +9,5 @@
   <!-- arm -->
   <xacro:ur5_robot prefix="" joint_limited="true"
-    shoulder_pan_lower_limit="${-pi}" shoulder_pan_upper_limit="${pi}"
+    shoulder_pan_lower_limit="${-2.4}" shoulder_pan_upper_limit="${0.8}"
     shoulder_lift_lower_limit="${-pi}" shoulder_lift_upper_limit="${pi}"
     elbow_joint_lower_limit="${-pi}" elbow_joint_upper_limit="${pi}"
@@ -17,9 +17,36 @@
     transmission_hw_interface="$(arg transmission_hw_interface)"
   />
+  <!-- gripper -->
+  <xacro:include filename="$(find ur5)/robotiq_description/urdf/robotiq_85_gripper.urdf.xacro" />
+  <xacro:robotiq_85_gripper prefix="" parent="ee_link" >
+	<origin xyz="0 0 0" rpy="${1.5708} 0 0" /> <!-- x must be greater than 0.004 -->
+  </xacro:robotiq_85_gripper>
+  <!-- A ground plane -->
+  <include>
+    <uri>model://ground_plane</uri>
+    <pose>0 0 0 0 0 0</pose>
+  </include>
+  <!-- base -->
+  <xacro:include filename="$(find ur5)/urdf/base.urdf" />
+  <xacro:base_ur5 parent="world" >
+	<origin xyz="-1 0.425 ${-0.1-0.955}" rpy="${1.5708} 0 ${1.5708*0.5} " />
+  </xacro:base_ur5>
+  <!-- camerabase -->
+  <xacro:include filename="$(find ur5)/urdf/camera_mount.urdf" />
+  <xacro:camera_mount parent="ee_link" >
+	<origin xyz="${0.01} ${-(0.3-0.3+0.05)} 0" rpy="0 ${1.5708*2} 0" />
+<!-- change x{0} value for position -->
+  </xacro:camera_mount>
+  <!-- camera -->
+  <xacro:include filename="$(find ur5)/urdf/camera.xacro" />
+  <xacro:camera parent="ee_link" >
+	<origin xyz="${-0.005+0.01} ${-0.08} ${-0.025}" rpy="${-1.5708} ${-1.5708} 0" />
+<!-- change x{0} value for position -->
+  </xacro:camera>
   <link name="world" />
   <joint name="world_joint" type="fixed">
     <parent link="world" />
     <child link = "base_link" />
-    <origin xyz="0.0 0.0 0" rpy="0.0 0.0 0.0" />
+    <origin xyz="0.0 0.0 0.0" rpy="0 0 0" />
   </joint>
 </robot>

File: ur5/urdf/ur5_robot.urdf.xacro (robot description, xacro)
@@ -13,5 +13,5 @@
   <xacro:include filename="$(find ur5)/robotiq_description/urdf/robotiq_85_gripper.urdf.xacro" />
   <xacro:robotiq_85_gripper prefix="" parent="ee_link" >
-	<origin xyz="0.005 0 0" rpy="${1.5708} 0 0" /> <!-- x must be greater than 0.004 -->
+	<origin xyz="0 0 0" rpy="${1.5708} 0 0" /> <!-- x must be greater than 0.004 -->
   </xacro:robotiq_85_gripper>
   <!-- A ground plane -->
@@ -23,10 +23,10 @@
   <xacro:include filename="$(find ur5)/urdf/base.urdf" />
   <xacro:base_ur5 parent="world" >
-	<origin xyz="-0.4 1 -0.1" rpy="${1.5708} 0 0 " />
+	<origin xyz="-1 0.425 ${-0.1-0.955}" rpy="${1.5708} 0 ${1.5708*0.5} " />
   </xacro:base_ur5>
   <!-- camerabase -->
   <xacro:include filename="$(find ur5)/urdf/camera_mount.urdf" />
   <xacro:camera_mount parent="ee_link" >
-	<origin xyz="${0} ${-(0.3-0.3+0.06)} 0" rpy="0 ${1.5708*2} 0" />
+	<origin xyz="${0.01} ${-(0.3-0.3+0.05)} 0" rpy="0 ${1.5708*2} 0" />
 <!-- change x{0} value for position -->
   </xacro:camera_mount>
@@ -34,5 +34,5 @@
   <xacro:include filename="$(find ur5)/urdf/camera.xacro" />
   <xacro:camera parent="ee_link" >
-	<origin xyz="${-0.005+0} ${-0.09} ${-0.025}" rpy="${-1.5708} ${-1.5708} 0" />
+	<origin xyz="${-0.005+0.01} ${-0.08} ${-0.025}" rpy="${-1.5708} ${-1.5708} 0 " />
 <!-- change x{0} value for position -->
   </xacro:camera>
@@ -41,5 +41,5 @@
     <parent link="world" />
     <child link = "base_link" />
-    <origin xyz="0.0 0.0 0.955" rpy="0 0 ${-1.5708*0.5}" />
+    <origin xyz="0.0 0.0 0.0" rpy="0 0 0" />
   </joint>
 </robot>
